File: BitFit/MainBoard v1.0.brd (EAGLE design)
At the start: 32.5 x 10.5 mm, 26 parts, among them J1 MICROUSB, U1 ATMEGA32U2QFN, U2 MCP738312, U3 LIS331, U5 REGULATOR

Commit message: Version 1.0
Finished version 1.0 of layout.
Parts:
- removed R10: (no value), BitFit:R0402
- removed U$11: LED_0402, BitFit:R0402
- added C3: 4.7uF, BitFit:C0402
- moved U$10 17.6 mm to (30.6, 1.00), turned to 180 degrees
- moved R2 13.3 mm to (14.6, 1.80)
- moved R3 12.5 mm to (12.4, 1.00)
- moved R4 11.5 mm to (21.3, 1.70), flipped to the bottom
- moved U3 9.68 mm to (27.4, 7.59)
- moved R5 7.91 mm to (24.0, 1.70), flipped to the bottom, turned to 0 degrees
- moved R9 7.90 mm to (13.0, 9.64), flipped to the bottom, turned to 180 degrees
- moved R11 6.44 mm to (17.6, 7.40), turned to 180 degrees
- moved R6 4.44 mm to (26.7, 1.70), flipped to the bottom
- moved U1 2.95 mm to (22.2, 4.00), turned to 0 degrees
- moved R7 1.52 mm to (29.4, 1.70), flipped to the bottom
- moved J1 1.30 mm to (5.40, 0.00)
- moved U$4 1.17 mm to (30.6, 8.25), turned to 0 degrees
- moved U$5 0.78 mm to (30.6, 6.25), turned to 0 degrees
- moved R1 0.41 mm to (19.7, 7.80)
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Connections:
- removed net N$24: U1.20, U3.9
- removed net N$28: U$4.2, U1.26
- new net N$31: R7.1, U1.9
- net +3V3: now also C3.1, R11.1, U1.27
- net +5V: no longer U$11.2
- net GND: now also C3.2, U$4.1, U$5.1, U$6.1, U$7.1; no longer R10.2, R11.1, R4.2, R5.2, R6.2, R7.2
- net N$15: now also U1.12, U3.11; no longer R10.1, U$11.1
- net N$16: now also R4.1, U1.18; no longer A1.P$31, U1.9
- net N$17: now also R6.1, U1.10; no longer A1.P$30, U1.8
- net N$20: now also R5.1, U1.11; no longer A1.P$33, U1.7
- net N$23: now also U1.13, U3.9; no longer U1.19, U3.11
- net N$25: now also A1.P$31, U1.26; no longer U$7.2, U1.22
- net N$26: now also A1.P$30, U1.22; no longer U$6.2, U1.23
- net N$27: now also A1.P$33; no longer U$5.2
- net N$4: now also R4.2, U$4.2; no longer R4.1, U$4.1
- net N$5: now also R5.2, U$5.2; no longer R5.1, U$5.1
- net N$6: now also R6.2, U$6.2; no longer R6.1, U$6.1
- net N$7: now also R7.2, U$7.2; no longer R7.1, U$7.1
Routing:
- net +3V3: track 3.62 -> 57.8 mm, vias 0 -> 5
- net +5V: track 4.49 -> 31.7 mm, vias 0 -> 2
- net N$14: track 0.00 -> 26.5 mm, vias 0 -> 1
- net GND: track 6.51 -> 28.2 mm, vias 1 -> 6
- net N$4: track 0.00 -> 14.6 mm, vias 0 -> 1
- net N$5: track 0.00 -> 12.6 mm, vias 0 -> 1
- net N$26: track 0.00 -> 9.61 mm, vias 0 -> 2
- net N$1: track 0.00 -> 8.50 mm, vias 0 -> 1
- net N$16: track 0.00 -> 8.17 mm, vias 0 -> 1
- net N$6: track 0.00 -> 8.15 mm, vias 0 -> 1
- net N$15: track 0.00 -> 8.02 mm
- net N$25: track 0.00 -> 7.11 mm
- net N$31: track 0.00 -> 6.92 mm, vias 0 -> 1
- net N$27: track 0.00 -> 5.90 mm
- net N$22: track 0.00 -> 5.65 mm, vias 0 -> 2
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- removed copper zone on layer 16, net GND
