File: BitFit/MainBoard v1.0.sch (EAGLE design)
At the start: 26 parts, among them J1 MICROUSB, U1 ATMEGA32U2QFN, U2 MCP738312, U3 LIS331, U5 REGULATOR

Commit message: Version 1.0
Finished version 1.0 of layout.
Parts:
- removed R10: (no value), BitFit:R-US_R0402
- removed U$11: LED_0402, BitFit:LED_0402
- added C3: 4.7uF, BitFit:C-USC0402
Connections:
- removed net N$24: U1.PB6, U3.INT2
- removed net N$28: U$4.P2, U1.PC4
- new net N$31: R7.1, U1.PD3
- net +3V3: now also C3.1, R11.1, U1.UCAP
- net +5V: no longer U$11.P2
- net GND: now also C3.2, U$4.P1, U$5.P1, U$6.P1, U$7.P1; no longer R10.2, R11.1, R4.2, R5.2, R6.2, R7.2
- net N$15: now also U1.PD6, U3.INT1; no longer R10.1, U$11.P1
- net N$16: now also R4.1, U1.PB4; no longer A1.PO_2(RX), U1.PD3
- net N$17: now also R6.1, U1.PD4; no longer A1.PO_3(TX), U1.PD2
- net N$20: now also R5.1, U1.PD5; no longer A1.PO_0, U1.PD1
- net N$23: now also U1.PD7, U3.INT2; no longer U1.PB5, U3.INT1
- net N$25: now also A1.PO_2(RX), U1.PC4; no longer U$7.P2, U1.PC7
- net N$26: now also A1.PO_3(TX), U1.PC7; no longer U$6.P2, U1.PC6
- net N$27: now also A1.PO_0; no longer U$5.P2
- net N$4: now also R4.2, U$4.P2; no longer R4.1, U$4.P1
- net N$5: now also R5.2, U$5.P2; no longer R5.1, U$5.P1
- net N$6: now also R6.2, U$6.P2; no longer R6.1, U$6.P1
- net N$7: now also R7.2, U$7.P2; no longer R7.1, U$7.P1
Other:
- moved on the sheet: A1, R11, R2, R3, R4, R5, R6, R7, U$4, U$5, U$6, U$7
