File: BitFit/MainBoard.brd (EAGLE design)
At the start: 32.5 x 10.5 mm, 6 parts, among them U1 MMA8452Q

Commit message: Version 1.0
Finished version 1.0 of layout.
Parts:
- removed ATMEGA: ATMEGA32U2QFN, BitFit:QFN-32
- removed U$1: MICROUSB, BitFit:MICROUSB
- removed U$3: LI-POL_BAT, BitFit:LI-POLY_28
- added BT: LI-POL_BAT, BitFit:LI-POLY_28
- added C1, C2: 4.7uF, BitFit:C0402
- added J1: MICROUSB, BitFit:MICROUSB
- added R10, R11, R2, R3, R4, R5, R6, R7, R9: (no value), BitFit:R0402
- added R8: 67K, BitFit:R0402
- added U$10, U$11, U$4, U$5, U$6, U$7: LED_0402, BitFit:R0402
- added U2: MCP738312, BitFit:SOT23-5
- added U3: LIS331, SparkFun-Sensors:LGA16-3MM
- added U5: REGULATOR, BitFit:SOT23-3
- U1: value MMA8452Q -> ATMEGA32U2QFN; device SparkFun-Sensors:QFN-16_0.5MM -> BitFit:QFN-32
- moved R1 6.05 mm to (15.0, 14.4), turned to 270 degrees
- moved U1 3.77 mm to (22.0, 4.00)
- renumbered U$2 to A1
Connections:
- removed net VDD: A1.P$17, A1.P$8, ATMEGA.31, ATMEGA.32, ATMEGA.4, U$1.VCC, U$3.VDD
- new net +3V3: A1.P$17, A1.P$8, U1.32, U1.4, U3.1, U3.14, U3.15, U5.2
- new net +5V: C2.1, J1.VCC, U$10.2, U$11.2, U1.31, U2.4
- new net N$10: BT.VDD, C1.1, U2.3, U5.3
- new net N$11: A1.P$34, R11.2
- new net N$12: R8.1, U2.5
- new net N$13: R9.1, U2.1
- new net N$14: R9.2, U$10.1
- new net N$15: R10.1, U$11.1
- new net N$16: U1.9
- new net N$17: U1.8
- new net N$18: U1.15, U3.4
- new net N$19: U1.14, U3.8
- new net N$20: U1.7
- new net N$21: U1.16, U3.6
- new net N$22: U1.17, U3.7
- new net N$23: U1.19, U3.11
- new net N$24: U1.20, U3.9
- new net N$25: A1.P$31, U1.26
- new net N$26: A1.P$30, U1.22
- new net N$27: A1.P$33, U1.25
- new net N$28: U1.1, U1.27
- new net N$4: R4.1, U$4.1
- new net N$5: R5.1, U$5.1
- new net N$6: R6.1, U$6.1
- new net N$7: R7.1, U$7.1
- new net N$8: J1.D+, R3.1
- new net N$9: J1.D-, R2.1
- net GND: now also BT.GND, C1.2, C2.2, J1.GND, R10.2, R11.1, R4.2, R5.2, R6.2, R7.2, R8.2, U1.28, U1.3, U2.2, U3.10, U3.12, U3.13, U3.16, U3.5, U5.1; no longer ATMEGA.28, ATMEGA.3, U$1.GND, U$3.GND
- net N$1: now also R3.2, U1.29; no longer ATMEGA.29, U$1.D+
- net N$2: now also R2.2, U1.30; no longer ATMEGA.30, U$1.D-
- net N$3: now also U1.24; no longer ATMEGA.24
Routing:
- net +3V3: track 0.00 -> 21.3 mm, vias 0 -> 1
- net GND: track 0.00 -> 13.5 mm, vias 0 -> 4
- net N$10: track 0.00 -> 9.49 mm
- net N$9: track 0.00 -> 8.97 mm
- net N$8: track 0.00 -> 8.66 mm
- net N$1: track 0.00 -> 8.56 mm, vias 0 -> 1
- net N$26: track 0.00 -> 8.18 mm, vias 0 -> 2
- net N$25: track 0.00 -> 5.39 mm
- net N$2: track 0.00 -> 5.31 mm, vias 0 -> 1
- net N$27: track 0.00 -> 4.94 mm
- net +5V: track 0.00 -> 4.12 mm
- net N$11: track 0.00 -> 2.15 mm
- net N$12: track 0.00 -> 1.60 mm
- added copper zone on layer 16, net +3V3
- added copper zone on layer 1, net GND
