File: BitFit/MainBoard v1.2.sch (EAGLE design)
At the start: 25 parts, among them J1 MICROUSB, U1 ATMEGA32U2QFN, U2 MCP738312, U3 LIS331, U5 REGULATOR

Commit message: File Clean Up v2
Parts:
- R4, R5, R6, R7, R9: value (none) -> 220ohm
- renumbered U$10 to L5, U$4 to L1, U$5 to L2, U$6 to L3, U$7 to L4
Connections:
- new net N$33: C3.1, U1.UCAP
- net +5V: no longer C3.1, U1.UCAP
Changed lines of the file:
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@@
 <?xml version="1.0" encoding="utf-8"?>
 <!DOCTYPE eagle SYSTEM "eagle.dtd">
-<eagle version="7.2.0">
+<eagle version="7.0.0">
 <drawing>
 <settings>
@@
 <part name="R2" library="BitFit" deviceset="R-US_" device="R0402" value="22ohm"/>
 <part name="R3" library="BitFit" deviceset="R-US_" device="R0402" value="22ohm"/>
-<part name="U$4" library="BitFit" deviceset="LED_0402" device=""/>
-<part name="U$5" library="BitFit" deviceset="LED_0402" device=""/>
-<part name="U$6" library="BitFit" deviceset="LED_0402" device=""/>
-<part name="U$7" library="BitFit" deviceset="LED_0402" device=""/>
-<part name="R4" library="BitFit" deviceset="R-US_" device="R0402"/>
-<part name="R5" library="BitFit" deviceset="R-US_" device="R0402"/>
-<part name="R6" library="BitFit" deviceset="R-US_" device="R0402"/>
-<part name="R7" library="BitFit" deviceset="R-US_" device="R0402"/>
+<part name="L1" library="BitFit" deviceset="LED_0402" device=""/>
+<part name="L2" library="BitFit" deviceset="LED_0402" device=""/>
+<part name="L3" library="BitFit" deviceset="LED_0402" device=""/>
+<part name="L4" library="BitFit" deviceset="LED_0402" device=""/>
+<part name="R4" library="BitFit" deviceset="R-US_" device="R0402" value="220ohm"/>
+<part name="R5" library="BitFit" deviceset="R-US_" device="R0402" value="220ohm"/>
+<part name="R6" library="BitFit" deviceset="R-US_" device="R0402" value="220ohm"/>
+<part name="R7" library="BitFit" deviceset="R-US_" device="R0402" value="220ohm"/>
 <part name="P+1" library="supply1" deviceset="+5V" device=""/>
 <part name="+3V2" library="supply1" deviceset="+3V3" device=""/>
@@
 <part name="U3" library="SparkFun-Sensors" deviceset="LIS331" device=""/>
 <part name="U2" library="BitFit" deviceset="MCP738312" device=""/>
-<part name="U$10" library="BitFit" deviceset="LED_0402" device=""/>
-<part name="R9" library="BitFit" deviceset="R-US_" device="R0402"/>
+<part name="L5" library="BitFit" deviceset="LED_0402" device=""/>
+<part name="R9" library="BitFit" deviceset="R-US_" device="R0402" value="220ohm"/>
 <part name="GND10" library="BitFit" deviceset="GND" device=""/>
 <part name="R11" library="BitFit" deviceset="R-US_" device="R0402"/>
@@
 <part name="GND2" library="BitFit" deviceset="GND" device=""/>
 <part name="+3V5" library="supply1" deviceset="+3V3" device=""/>
-<part name="P+3" library="supply1" deviceset="+5V" device=""/>
 <part name="GND7" library="BitFit" deviceset="GND" device=""/>
 <part name="GND6" library="BitFit" deviceset="GND" device=""/>
@@
 <instance part="R2" gate="G$1" x="25.4" y="53.34"/>
 <instance part="R3" gate="G$1" x="43.18" y="55.88"/>
-<instance part="U$4" gate="G$1" x="154.94" y="88.9"/>
-<instance part="U$5" gate="G$1" x="154.94" y="96.52"/>
-<instance part="U$6" gate="G$1" x="154.94" y="104.14"/>
-<instance part="U$7" gate="G$1" x="154.94" y="111.76"/>
+<instance part="L1" gate="G$1" x="154.94" y="88.9"/>
+<instance part="L2" gate="G$1" x="154.94" y="96.52"/>
+<instance part="L3" gate="G$1" x="154.94" y="104.14"/>
+<instance part="L4" gate="G$1" x="154.94" y="111.76"/>
 <instance part="R4" gate="G$1" x="137.16" y="88.9"/>
 <instance part="R5" gate="G$1" x="137.16" y="96.52"/>
@@
 <instance part="U3" gate="G$1" x="144.78" y="58.42" rot="MR0"/>
 <instance part="U2" gate="G$1" x="-93.98" y="55.88" rot="R180"/>
-<instance part="U$10" gate="G$1" x="-104.14" y="71.12"/>
+<instance part="L5" gate="G$1" x="-104.14" y="71.12"/>
 <instance part="R9" gate="G$1" x="-88.9" y="71.12" rot="R180"/>
 <instance part="GND10" gate="1" x="-73.66" y="68.58"/>
@@
 <instance part="GND2" gate="1" x="33.02" y="83.82" rot="R180"/>
 <instance part="+3V5" gate="G$1" x="167.64" y="33.02" rot="MR0"/>
-<instance part="P+3" gate="1" x="33.02" y="58.42" rot="R180"/>
 <instance part="GND7" gate="1" x="-7.62" y="48.26"/>
 <instance part="GND6" gate="1" x="172.72" y="81.28"/>
@@
 <wire x1="-119.38" y1="78.74" x2="-119.38" y2="83.82" width="0.1524" layer="91"/>
 <wire x1="-119.38" y1="60.96" x2="-109.22" y2="60.96" width="0.1524" layer="91"/>
-<pinref part="U$10" gate="G$1" pin="P2"/>
+<pinref part="L5" gate="G$1" pin="P2"/>
 <wire x1="-111.76" y1="71.12" x2="-119.38" y2="71.12" width="0.1524" layer="91"/>
 <junction x="-119.38" y="71.12"/>
@@
 <wire x1="40.64" y1="83.82" x2="40.64" y2="78.74" width="0.1524" layer="91"/>
 <wire x1="40.64" y1="78.74" x2="53.34" y2="78.74" width="0.1524" layer="91"/>
-</segment>
-<segment>
-<pinref part="U1" gate="G$1" pin="UCAP"/>
-<pinref part="C3" gate="G$1" pin="1"/>
-<wire x1="53.34" y1="60.96" x2="40.64" y2="60.96" width="0.1524" layer="91"/>
-<wire x1="40.64" y1="60.96" x2="40.64" y2="63.5" width="0.1524" layer="91"/>
-<wire x1="40.64" y1="63.5" x2="33.02" y2="63.5" width="0.1524" layer="91"/>
-<wire x1="33.02" y1="63.5" x2="33.02" y2="60.96" width="0.1524" layer="91"/>
-<wire x1="33.02" y1="63.5" x2="33.02" y2="66.04" width="0.1524" layer="91"/>
-<pinref part="P+3" gate="1" pin="+5V"/>
 </segment>
 </net>
@@
 <segment>
 <wire x1="172.72" y1="88.9" x2="172.72" y2="96.52" width="0.1524" layer="91"/>
-<pinref part="U$4" gate="G$1" pin="P1"/>
+<pinref part="L1" gate="G$1" pin="P1"/>
 <wire x1="172.72" y1="96.52" x2="172.72" y2="104.14" width="0.1524" layer="91"/>
 <wire x1="172.72" y1="104.14" x2="172.72" y2="111.76" width="0.1524" layer="91"/>
 <wire x1="162.56" y1="88.9" x2="172.72" y2="88.9" width="0.1524" layer="91"/>
-<pinref part="U$5" gate="G$1" pin="P1"/>
+<pinref part="L2" gate="G$1" pin="P1"/>
 <wire x1="162.56" y1="96.52" x2="172.72" y2="96.52" width="0.1524" layer="91"/>
 <junction x="172.72" y="96.52"/>
-<pinref part="U$6" gate="G$1" pin="P1"/>
+<pinref part="L3" gate="G$1" pin="P1"/>
 <wire x1="162.56" y1="104.14" x2="172.72" y2="104.14" width="0.1524" layer="91"/>
 <junction x="172.72" y="104.14"/>
-<pinref part="U$7" gate="G$1" pin="P1"/>
+<pinref part="L4" gate="G$1" pin="P1"/>
 <wire x1="162.56" y1="111.76" x2="172.72" y2="111.76" width="0.1524" layer="91"/>
 <junction x="172.72" y="88.9"/>
@@
 <net name="N$14" class="0">
 <segment>
-<pinref part="U$10" gate="G$1" pin="P1"/>
+<pinref part="L5" gate="G$1" pin="P1"/>
 <pinref part="R9" gate="G$1" pin="2"/>
 <wire x1="-96.52" y1="71.12" x2="-93.98" y2="71.12" width="0.1524" layer="91"/>
@@
 <segment>
 <pinref part="R4" gate="G$1" pin="2"/>
-<pinref part="U$4" gate="G$1" pin="P2"/>
+<pinref part="L1" gate="G$1" pin="P2"/>
 <wire x1="142.24" y1="88.9" x2="147.32" y2="88.9" width="0.1524" layer="91"/>
 </segment>
@@
 <segment>
 <pinref part="R5" gate="G$1" pin="2"/>
-<pinref part="U$5" gate="G$1" pin="P2"/>
+<pinref part="L2" gate="G$1" pin="P2"/>
 <wire x1="142.24" y1="96.52" x2="147.32" y2="96.52" width="0.1524" layer="91"/>
 </segment>
@@
 <segment>
 <pinref part="R6" gate="G$1" pin="2"/>
-<pinref part="U$6" gate="G$1" pin="P2"/>
+<pinref part="L3" gate="G$1" pin="P2"/>
 <wire x1="142.24" y1="104.14" x2="147.32" y2="104.14" width="0.1524" layer="91"/>
 </segment>
@@
 <segment>
 <pinref part="R7" gate="G$1" pin="2"/>
-<pinref part="U$7" gate="G$1" pin="P2"/>
+<pinref part="L4" gate="G$1" pin="P2"/>
 <wire x1="142.24" y1="111.76" x2="147.32" y2="111.76" width="0.1524" layer="91"/>
 </segment>
@@
 </segment>
 </net>
+<net name="N$33" class="0">
+<segment>
+<pinref part="U1" gate="G$1" pin="UCAP"/>
+<pinref part="C3" gate="G$1" pin="1"/>
+<wire x1="53.34" y1="60.96" x2="40.64" y2="60.96" width="0.1524" layer="91"/>
+<wire x1="40.64" y1="60.96" x2="40.64" y2="63.5" width="0.1524" layer="91"/>
+<wire x1="33.02" y1="63.5" x2="33.02" y2="66.04" width="0.1524" layer="91"/>
+<wire x1="33.02" y1="63.5" x2="40.64" y2="63.5" width="0.1524" layer="91"/>
+</segment>
+</net>
